File: kicad/usb_soil_moisture.kicad_pcb (KiCad board)
At the start: 2 copper layers, 2 parts, among them U1 SeeeduinoXIAO, U2 SENO0193

Commit message: DRC ok
Parts:
- added ~: signature_koino, kicad_mylib:signature_koino, F.Cu at (7.62, -44.5)
- added ~: akizuki_C_plate, kicad_mylib:akizuki_C_plate, F.Cu at (0.00, 0.00)
Routing:
- net GND: track 64.9 -> 55.1 mm
- net +5V: track 56.6 -> 55.6 mm
- added copper zone on B.Cu, net GND
- added copper zone on F.Cu, net GND
Other:
- board outline added: 72 x 47.5 mm
Changed lines of the file:
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@@
     (thickness 1.6)
     (drawings 0)
-    (tracks 18)
+    (tracks 16)
     (zones 0)
-    (modules 2)
+    (modules 4)
     (nets 21)
   )
@@
     (pcbplotparams
       (layerselection 0x010fc_ffffffff)
-      (usegerberextensions false)
+      (usegerberextensions true)
       (usegerberattributes false)
       (usegerberadvancedattributes false)
@@
       (outputformat 1)
       (mirror false)
-      (drillshape 1)
+      (drillshape 0)
       (scaleselection 1)
-      (outputdirectory ""))
+      (outputdirectory "gerbers/"))
   )
   (net 0 "")
@@
     (add_net "Net-(U1-Pad9)")
   )
+  (module kicad_mylib:signature_koino (layer F.Cu)
+    (at 7.62 -44.45)
+    (fp_text reference ~ (at 2.54 -3.81) (layer F.SilkS)
+      (effects (font (size 1 1) (thickness 0.15)))
+    )
+    (fp_text value signature_koino (at 6.35 -5.58) (layer F.Fab)
+      (effects (font (size 1 1) (thickness 0.15)))
+    )
+    (fp_text user "Twitter:@koino_mfg  USB-SOIL-MOISTURE" (at 0 -1.27) (layer F.SilkS)
+      (effects (font (size 1 1) (thickness 0.15)) (justify left))
+    )
+  )
+  (module kicad_mylib:akizuki_C_plate (layer F.Cu)
+    (at 0 0)
+    (fp_text reference ~ (at 6.35 -49.03) (layer F.SilkS)
+      (effects (font (size 1 1) (thickness 0.15)))
+    )
+    (fp_text value akizuki_C_plate (at 6.35 -50.03) (layer F.Fab)
+      (effects (font (size 1 1) (thickness 0.15)))
+    )
+    (fp_line (start 72 -32.64) (end 72 -44.96) (layer Edge.Cuts) (width 0.12))
+    (fp_line (start 62 -32.64) (end 72 -32.64) (layer Edge.Cuts) (width 0.12))
+    (fp_line (start 62 -14.86) (end 72 -14.86) (layer Edge.Cuts) (width 0.12))
+    (fp_line (start 62 -32.64) (end 62 -14.86) (layer Edge.Cuts) (width 0.12))
+    (fp_circle (center 69 -44.5) (end 70.6 -44.5) (layer Edge.Cuts) (width 0.12))
+    (fp_circle (center 69 -3) (end 70.6 -3) (layer Edge.Cuts) (width 0.12))
+    (fp_circle (center 3 -44.5) (end 4.6 -44.5) (layer Edge.Cuts) (width 0.12))
+    (fp_circle (center 3 -3) (end 4.6 -3) (layer Edge.Cuts) (width 0.12))
+    (fp_arc (start 69.46 -44.96) (end 72 -44.96) (angle -90) (layer Edge.Cuts) (width 0.12))
+    (fp_line (start 72 -2.54) (end 72 -14.86) (layer Edge.Cuts) (width 0.12))
+    (fp_line (start 2.54 -47.5) (end 69.46 -47.5) (layer Edge.Cuts) (width 0.12))
+    (fp_arc (start 2.54 -44.96) (end 2.54 -47.5) (angle -90) (layer Edge.Cuts) (width 0.12))
+    (fp_line (start 0 -2.54) (end 0 -44.96) (layer Edge.Cuts) (width 0.12))
+    (fp_arc (start 69.46 -2.54) (end 69.46 0) (angle -90) (layer Edge.Cuts) (width 0.12))
+    (fp_line (start 2.54 0) (end 69.46 0) (layer Edge.Cuts) (width 0.12))
+    (fp_arc (start 2.54 -2.54) (end 0 -2.54) (angle -90) (layer Edge.Cuts) (width 0.12))
+  )
   (module kicad_mylib:SENO0193 (layer F.Cu)
     (at 6.35 -20.32)
-    (fp_text reference U2 (at 1.27 -9.66) (layer F.SilkS)
+    (fp_text reference U2 (at 0 1.27) (layer F.SilkS)
       (effects (font (size 1 1) (thickness 0.15)))
     )
@@
       (effects (font (size 1 1) (thickness 0.15)))
     )
-    (fp_text user REF** (at 1.27 -8.89) (layer F.SilkS)
+    (fp_text user SENO0193 (at 1.27 -8.89) (layer F.SilkS)
       (effects (font (size 1 1) (thickness 0.15)))
     )
@@
     (at 40.94 -32.62 270)
     (attr smd)
-    (fp_text reference U1 (at 9.3345 -21.7805 90) (layer F.SilkS)
+    (fp_text reference U1 (at 9.3345 1.57 90) (layer F.SilkS)
       (effects (font (size 0.889 0.889) (thickness 0.1016)))
     )
@@
       (net 14 "Net-(U1-Pad8)"))
   )
+  (segment (start 59.05782 -31.78688) (end 59.05782 -32.16153) (width 0.25) (layer F.Cu) (net 7))
   (segment (start 59.05782 -32.16153) (end 56.92935 -34.29) (width 0.25) (layer F.Cu) (net 7))
-  (segment (start 59.05782 -31.78688) (end 59.05782 -32.16153) (width 0.25) (layer F.Cu) (net 7))
-  (segment (start 56.92935 -34.29) (end 19.05 -34.29) (width 0.25) (layer F.Cu) (net 7))
-  (segment (start 11.43 -26.67) (end 7.62 -26.67) (width 0.25) (layer F.Cu) (net 7))
-  (segment (start 19.05 -34.29) (end 11.43 -26.67) (width 0.25) (layer F.Cu) (net 7))
-  (segment (start 21.59 -11.43) (end 11.43 -21.59) (width 0.25) (layer F.Cu) (net 19))
-  (segment (start 57.15 -11.43) (end 21.59 -11.43) (width 0.25) (layer F.Cu) (net 19))
-  (segment (start 60.38232 -14.66232) (end 57.15 -11.43) (width 0.25) (layer F.Cu) (net 19))
-  (segment (start 60.38232 -16.545595) (end 60.38232 -14.66232) (width 0.25) (layer F.Cu) (net 19))
-  (segment (start 59.606445 -17.32147) (end 60.38232 -16.545595) (width 0.25) (layer F.Cu) (net 19))
-  (segment (start 11.43 -21.59) (end 7.62 -21.59) (width 0.25) (layer F.Cu) (net 19))
-  (segment (start 57.83847 -17.32147) (end 59.606445 -17.32147) (width 0.25) (layer F.Cu) (net 19))
-  (segment (start 56.517 -16) (end 57.83847 -17.32147) (width 0.25) (layer F.Cu) (net 19))
-  (segment (start 57.73332 -13.92317) (end 21.63683 -13.92317) (width 0.25) (layer F.Cu) (net 20))
-  (segment (start 59.05782 -15.24767) (end 57.73332 -13.92317) (width 0.25) (layer F.Cu) (net 20))
+  (segment (start 56.92935 -34.29) (end 21.59 -34.29) (width 0.25) (layer F.Cu) (net 7))
+  (segment (start 13.97 -26.67) (end 7.62 -26.67) (width 0.25) (layer F.Cu) (net 7))
+  (segment (start 21.59 -34.29) (end 13.97 -26.67) (width 0.25) (layer F.Cu) (net 7))
+  (segment (start 56.51782 -13.33782) (end 56.51782 -15.62232) (width 0.25) (layer F.Cu) (net 19))
+  (segment (start 55.88 -12.7) (end 56.51782 -13.33782) (width 0.25) (layer F.Cu) (net 19))
+  (segment (start 13.97 -21.59) (end 22.86 -12.7) (width 0.25) (layer F.Cu) (net 19))
+  (segment (start 22.86 -12.7) (end 55.88 -12.7) (width 0.25) (layer F.Cu) (net 19))
+  (segment (start 7.62 -21.59) (end 13.97 -21.59) (width 0.25) (layer F.Cu) (net 19))
   (segment (start 59.05782 -15.62232) (end 59.05782 -15.24767) (width 0.25) (layer F.Cu) (net 20))
-  (segment (start 11.43 -24.13) (end 7.62 -24.13) (width 0.25) (layer F.Cu) (net 20))
-  (segment (start 21.63683 -13.92317) (end 11.43 -24.13) (width 0.25) (layer F.Cu) (net 20))
+  (segment (start 7.62 -24.13) (end 13.97 -24.13) (width 0.25) (layer F.Cu) (net 20))
+  (segment (start 13.97 -24.13) (end 20.32 -17.78) (width 0.25) (layer F.Cu) (net 20))
+  (segment (start 59.05782 -15.99697) (end 59.05782 -15.62232) (width 0.25) (layer F.Cu) (net 20))
+  (segment (start 57.27479 -17.78) (end 59.05782 -15.99697) (width 0.25) (layer F.Cu) (net 20))
+  (segment (start 20.32 -17.78) (end 57.27479 -17.78) (width 0.25) (layer F.Cu) (net 20))
+  (zone (net 19) (net_name GND) (layer F.Cu) (hatch edge 0.508)
+    (connect_pads (clearance 0.508))
+    (min_thickness 0.254)
+    (fill yes (arc_segments 32) (thermal_gap 0.508) (thermal_bridge_width 0.508))
+    (polygon
+      (pts
+        (xy 73.66 -52.07) (xy -1.27 -52.07) (xy -1.27 3.81) (xy 73.66 3.81)
+      )
+    )
+  )
+  (zone (net 19) (net_name GND) (layer B.Cu) (hatch edge 0.508)
+    (connect_pads (clearance 0.508))
+    (min_thickness 0.254)
+    (fill yes (arc_segments 32) (thermal_gap 0.508) (thermal_bridge_width 0.508))
+    (polygon
+      (pts
+        (xy 76.2 -49.53) (xy -3.81 -49.53) (xy -3.81 1.27) (xy 76.2 1.27)
+      )
+    )
+  )
 )
